Commit message: gazebo模型可用

File: src/racecar_description/urdf/macros.xacro (robot description, xacro)
@@ -1,4 +1,4 @@
 <?xml version="1.0"?>
-<robot name="racebot" xmlns:xacro="http://www.ros.org/wiki/xacro">
+<robot name="racecar" xmlns:xacro="http://www.ros.org/wiki/xacro">
 <!-- transmission macros -->
 <!-- <xacro:macro name="wheel_transmission" params="name">

File: src/racecar_description/urdf/racecar.xacro (robot description, xacro)
@@ -1,5 +1,5 @@
 <?xml version="1.0" encoding="utf-8"?>
-<robot name="racebot" xmlns:xacro="http://www.ros.org/wiki/xacro">
-    <xacro:include filename="$(find racebot_description)/urdf/macros.xacro" />
+<robot name="racecar" xmlns:xacro="http://www.ros.org/wiki/xacro">
+    <xacro:include filename="$(find racecar_description)/urdf/macros.xacro" />
     <link name="base_footprint">
     </link>
@@ -7,5 +7,5 @@
         <visual>
             <geometry>
-                <box size="0.28 0.1 0.03"/>
+                <box size="2.8 1.0 0.3"/>
             </geometry>
             <origin xyz="0 0 0" rpy="0 0 0" />
@@ -16,5 +16,5 @@
         <collision>
             <geometry>
-                <box size="0.28 0.1 0.03" />
+                <box size="2.8 1.0 0.3" />
             </geometry>
             <origin xyz="0.0 0.0 0.0" rpy="0.0 0.0 0.0" />
@@ -23,5 +23,5 @@
             <origin xyz="0 0 0" />
             <mass value="4" />
-            <inertia ixx="0.0264" ixy="0" ixz="0" iyy="0.0294" iyz="0" izz="0.00364" />
+            <inertia ixx="264" ixy="0" ixz="0" iyy="294" iyz="0" izz="36.4" />
         </inertial>
     </link>
@@ -29,10 +29,10 @@
         <parent link="base_footprint" />
         <child link="base_link"/>
-        <origin xyz="0 0 0.032" />
+        <origin xyz="0 0 0.32" />
     </joint>
        <link name="left_steering_hinge">
         <visual>
             <geometry>
-                <cylinder radius="0.01" length="0.005" />
+                <cylinder radius="0.1" length="0.05" />
                 <!-- <sphere radius="0.015" /> -->
             </geometry>
@@ -44,5 +44,5 @@
         <collision>
             <geometry>
-                <cylinder radius="0.01" length="0.005" />
+                <cylinder radius="0.1" length="0.05" />
                 <!-- <sphere radius="0.015" /> -->
             </geometry>
@@ -52,5 +52,5 @@
             <origin xyz="0 0 0" />
             <mass value="1" />
-            <inertia ixx="2.7E-05" ixy="0" ixz="0" iyy="2.7E-05" iyz="0" izz="5E-05" />
+            <inertia ixx="2.7E-02" ixy="0" ixz="0" iyy="2.7E-02" iyz="0" izz="5E-02" />
         </inertial>
     </link>
@@ -58,28 +58,28 @@
         <parent link="base_link" />
         <child link="left_steering_hinge" />
-        <origin xyz="0.13 0.065 0" />
+        <origin xyz="1.3 0.65 0" />
         <axis xyz="0 0 1" />
-        <limit lower="-0.6" upper="0.6" effort="2.0" velocity="100.0"/>
+        <limit lower="-0.6" upper="0.6" effort="5" velocity="100.0"/>
     </joint>
     <link name="left_front_wheel">
         <visual>
             <geometry>
-                <cylinder radius="0.033" length="0.02" />
-            </geometry>
-            <origin xyz="0 0 0" rpy="1.57 0 0" />
-            <material name="black">
-                <color rgba="0.0 0.0 0.0 1.0" />
-            </material>
-        </visual>
-        <collision>
-            <geometry>
-                <cylinder radius="0.032" length="0.02" />
-            </geometry>
-            <origin xyz="0.0 0.0 0.0" rpy="1.57 0.0 0.0" />
-        </collision>
-        <inertial>
-            <origin xyz="0 0 0" />
-            <mass value="2.0" />
-            <inertia ixx="6.64E-04" ixy="0" ixz="0" iyy="6.64E-04" iyz="0" izz="1.02E-03" />
+                <cylinder radius="0.33" length="0.2" />
+            </geometry>
+            <origin xyz="0 0 0" rpy="1.57 0 0" />
+            <material name="black">
+                <color rgba="0.0 0.0 0.0 1.0" />
+            </material>
+        </visual>
+        <collision>
+            <geometry>
+                <cylinder radius="0.32" length="0.2" />
+            </geometry>
+            <origin xyz="0.0 0.0 0.0" rpy="1.57 0.0 0.0" />
+        </collision>
+        <inertial>
+            <origin xyz="0 0 0" />
+            <mass value="2" />
+            <inertia ixx="6.64E-01" ixy="0" ixz="0" iyy="6.64E-01" iyz="0" izz="1.02E+00" />
         </inertial>
     </link>
@@ -87,5 +87,5 @@
         <parent link="left_steering_hinge" />
         <child link="left_front_wheel" />
-        <origin xyz="0 0.025 0" />
+        <origin xyz="0 0.25 0" />
         <axis xyz="0 1 0" />
         <limit effort="10" velocity="1000" />
@@ -94,14 +94,14 @@
         <visual>
             <geometry>
-                 <cylinder radius="0.01" length="0.005" />
-            </geometry>
-            <origin xyz="0 0 0" rpy="1.57 0 0" />
-            <material name="black">
-                <color rgba="0.0 0.0 0.0 1.0" />
-            </material>
-        </visual>
-        <collision>
-            <geometry>
-                <cylinder radius="0.01" length="0.005" />
+                 <cylinder radius="0.1" length="0.05" />
+            </geometry>
+            <origin xyz="0 0 0" rpy="1.57 0 0" />
+            <material name="black">
+                <color rgba="0.0 0.0 0.0 1.0" />
+            </material>
+        </visual>
+        <collision>
+            <geometry>
+                <cylinder radius="0.1" length="0.05" />
             </geometry>
             <origin xyz="0.0 0.0 0.0" rpy="1.57 0.0 0.0" />
@@ -110,5 +110,5 @@
             <origin xyz="0 0 0" />
             <mass value="1" />
-            <inertia ixx="2.7E-05" ixy="0" ixz="0" iyy="2.7E-05" iyz="0" izz="5E-05" />
+            <inertia ixx="2.7E-02" ixy="0" ixz="0" iyy="2.7E-02" iyz="0" izz="5E-02" />
         </inertial>
     </link>
@@ -116,28 +116,28 @@
         <parent link="base_link" />
         <child link="right_steering_hinge" />
-        <origin xyz="0.13 -0.065 0" />
+        <origin xyz="1.3 -0.65 0" />
         <axis xyz="0 0 1" />
-        <limit lower="-0.6" upper="0.6" effort="2.0" velocity="100.0"/>
+        <limit lower="-0.6" upper="0.6" effort="5" velocity="100.0"/>
     </joint>
      <link name="right_front_wheel">
         <visual>
             <geometry>
-                <cylinder radius="0.033" length="0.02" />
-            </geometry>
-            <origin xyz="0 0 0" rpy="1.57 0 0" />
-            <material name="black">
-                <color rgba="0.0 0.0 0.0 1.0" />
-            </material>
-        </visual>
-        <collision>
-            <geometry>
-                <cylinder radius="0.032" length="0.02" />
-            </geometry>
-            <origin xyz="0.0 0.0 0.0" rpy="1.57 0.0 0.0" />
-        </collision>
-        <inertial>
-            <origin xyz="0 0 0" />
-            <mass value="2.0" />
-            <inertia ixx="6.64E-04" ixy="0" ixz="0" iyy="6.64E-04" iyz="0" izz="1.02E-03" />
+                <cylinder radius="0.33" length="0.2" />
+            </geometry>
+            <origin xyz="0 0 0" rpy="1.57 0 0" />
+            <material name="black">
+                <color rgba="0.0 0.0 0.0 1.0" />
+            </material>
+        </visual>
+        <collision>
+            <geometry>
+                <cylinder radius="0.32" length="0.2" />
+            </geometry>
+            <origin xyz="0.0 0.0 0.0" rpy="1.57 0.0 0.0" />
+        </collision>
+        <inertial>
+            <origin xyz="0 0 0" />
+            <mass value="2" />
+            <inertia ixx="6.64E-01" ixy="0" ixz="0" iyy="6.64E-01" iyz="0" izz="1.02E+00" />
         </inertial>
     </link>
@@ -145,5 +145,5 @@
         <parent link="right_steering_hinge" />
         <child link="right_front_wheel" />
-        <origin xyz="0 -0.025 0" />
+        <origin xyz="0 -0.25 0" />
         <axis xyz="0 1 0" />
         <limit effort="10" velocity="1000" />
@@ -152,21 +152,21 @@
         <visual>
             <geometry>
-                <cylinder radius="0.032" length="0.02" />
-            </geometry>
-            <origin xyz="0 0 0" rpy="1.57 0 0" />
-            <material name="black">
-                <color rgba="0.0 0.0 0.0 1.0" />
-            </material>
-        </visual>
-        <collision>
-            <geometry>
-                <cylinder radius="0.032" length="0.02" />
-            </geometry>
-            <origin xyz="0.0 0.0 0.0" rpy="1.57 0.0 0.0" />
-        </collision>
-        <inertial>
-            <origin xyz="0 0 0" />
-            <mass value="2.0" />
-            <inertia ixx="6.64E-04" ixy="0" ixz="0" iyy="6.64E-04" iyz="0" izz="1.02E-03" />
+                <cylinder radius="0.32" length="0.2" />
+            </geometry>
+            <origin xyz="0 0 0" rpy="1.57 0 0" />
+            <material name="black">
+                <color rgba="0.0 0.0 0.0 1.0" />
+            </material>
+        </visual>
+        <collision>
+            <geometry>
+                <cylinder radius="0.32" length="0.2" />
+            </geometry>
+            <origin xyz="0.0 0.0 0.0" rpy="1.57 0.0 0.0" />
+        </collision>
+        <inertial>
+            <origin xyz="0 0 0" />
+            <mass value="2" />
+            <inertia ixx="6.64E-01" ixy="0" ixz="0" iyy="6.64E-01" iyz="0" izz="1.02E+00" />
         </inertial>
     </link>
@@ -174,5 +174,5 @@
         <parent link="base_link" />
         <child link="left_rear_wheel" />
-        <origin xyz="-0.13 0.09 0" />
+        <origin xyz="-1.3 0.9 0" />
         <axis xyz="0 1 0" />
         <limit effort="10" velocity="1000" />
@@ -181,21 +181,21 @@
         <visual>
             <geometry>
-                <cylinder radius="0.032" length="0.02" />
-            </geometry>
-            <origin xyz="0 0 0" rpy="1.57 0 0" />
-            <material name="black">
-                <color rgba="0.0 0.0 0.0 1.0" />
-            </material>
-        </visual>
-        <collision>
-            <geometry>
-                <cylinder radius="0.032" length="0.02" />
-            </geometry>
-            <origin xyz="0.0 0.0 0.0" rpy="1.57 0.0 0.0" />
-        </collision>
-        <inertial>
-            <origin xyz="0 0 0" />
-            <mass value="2.0" />
-            <inertia ixx="6.64E-04" ixy="0" ixz="0" iyy="6.64E-04" iyz="0" izz="1.02E-03" />
+                <cylinder radius="0.32" length="0.2" />
+            </geometry>
+            <origin xyz="0 0 0" rpy="1.57 0 0" />
+            <material name="black">
+                <color rgba="0.0 0.0 0.0 1.0" />
+            </material>
+        </visual>
+        <collision>
+            <geometry>
+                <cylinder radius="0.32" length="0.2" />
+            </geometry>
+            <origin xyz="0.0 0.0 0.0" rpy="1.57 0.0 0.0" />
+        </collision>
+        <inertial>
+            <origin xyz="0 0 0" />
+            <mass value="2" />
+            <inertia ixx="6.64E-01" ixy="0" ixz="0" iyy="6.64E-01" iyz="0" izz="1.02E+00" />
         </inertial>
     </link>
@@ -203,8 +203,8 @@
         <parent link="base_link" />
         <child link="right_rear_wheel" />
-        <origin xyz="-0.13 -0.09 0" />
-        <axis xyz="0 1 0" />
-        <limit effort="10" velocity="1000" />
-    </joint>
-  <xacro:include filename="$(find racebot_description)/urdf/racecar.gazebo" />
+        <origin xyz="-1.3 -0.9 0" />
+        <axis xyz="0 1 0" />
+        <limit effort="10" velocity="1000" />
+    </joint>
+  <xacro:include filename="$(find racecar_description)/urdf/racecar.gazebo" />
 </robot>
